Commit message: add go2piper cfg

File: mani-centric-wbc/resources/robots/go2_piper/go2_piper.urdf (robot description, URDF)
Before this commit: robot go2piper, 44 links, 43 joints
Joints:
- joint joint7: axis 0 0 1 -> (none); limit lower=0 upper=0.035 effort=10 velocity=1 -> (none); type prismatic -> fixed
- joint joint8: axis 0 0 -1 -> (none); limit lower=-0.035 upper=0 effort=10 velocity=1 -> (none); type prismatic -> fixed
